Commit message: Add red and blue material

File: urdf/mira_simple.urdf (robot description, URDF)
Before this commit: robot mira, 2 links, 1 joints
Links:
- added link pitch_M2_link; visual cylinder length=0.01 radius=0.005
- added link yaw_M3_link; visual cylinder length=0.01 radius=0.005
Joints:
- added joint pitch_joint: type revolute, parent roll_M1_link, child pitch_M2_link, origin xyz=0.0 0.0 0.045 rpy=0 0 0, axis 1 0 0, limit lower=-0.2 upper=0.2 effort=0.1 velocity=0.005
- added joint yaw_joint: type revolute, parent pitch_M2_link, child yaw_M3_link, origin xyz=0.0 0.0 0.055 rpy=0 0 0, axis 1 0 0, limit lower=-0.2 upper=0.2 effort=0.1 velocity=0.005
- joint roll_joint: origin xyz=0.0023 0 -0.0005 rpy=0 0 0 -> xyz=0.0 0.0 0.045 rpy=0 0 0

Commit message: Correct roll pitch yaw links and joints

File: urdf/mira_simple.urdf (robot description, URDF)
Before this commit: robot mira, 4 links, 3 joints
Links:
- link pitch_M2_link: geometry visual cylinder length=0.005 radius=0.01
- link roll_M1_link: geometry visual cylinder length=0.005 radius=0.01
- link yaw_M3_link: geometry visual cylinder length=0.005 radius=0.01
Joints:
- joint pitch_joint: origin xyz=0.0 0.0 0.045 rpy=0 0 0 -> xyz=0.0 0.0 0.0025 rpy=0 0 0
- joint yaw_joint: origin xyz=0.0 0.0 0.055 rpy=0 0 0 -> xyz=0.0 0.0 0.0 rpy=0 0 0

Commit message: Add base_head_joint and head_link

File: urdf/mira_simple.urdf (robot description, URDF)
Before this commit: robot mira, 4 links, 3 joints
Links:
- added link head_link; visual sphere radius=0.06
Joints:
- added joint base_head_joint: type revolute, parent yaw_M3_link, child head_link, origin xyz=0.0 0.0 0.0 rpy=0 0 0, axis 1 0 0, limit lower=-0.2 upper=0.2 effort=0.1 velocity=0.005

Commit message: Add right and left eyes links and joints

File: urdf/mira_simple.urdf (robot description, URDF)
Before this commit: robot mira, 5 links, 4 joints
Links:
- added link left_eye_link; visual cylinder length=0.00525 radius=0.00525
- added link right_eye_link; visual cylinder length=0.00525 radius=0.00525
Joints:
- added joint head_lefteye_joint: type fixed, parent head_link, child left_eye_link, origin xyz=0.0470931 0.0271892 0.0253571 rpy=0 0 0
- added joint head_righteye_joint: type fixed, parent head_link, child right_eye_link, origin xyz=0.0470931 -0.0271892 0.0253571 rpy=0 0 0

Commit message: Add camera link and joint

File: urdf/mira_simple.urdf (robot description, URDF)
Before this commit: robot mira, 7 links, 6 joints
Links:
- added link camera_link; visual box size=0.0005 0.0005 0.0005
Joints:
- added joint head_camera_joint: type fixed, parent head_link, child camera_link, origin xyz=0.0424264 0 0.0424264 rpy=0 0 0

Commit message: Correct pitch yaw rotations

File: urdf/mira_simple.urdf (robot description, URDF)
Before this commit: robot mira, 8 links, 7 joints
Joints:
- joint pitch_joint: axis 1 0 0 -> 0 1 0
- joint yaw_joint: axis 1 0 0 -> 0 0 1

Commit message: Change base_head_joint to fixed

File: urdf/mira_simple.urdf (robot description, URDF)
Before this commit: robot mira, 8 links, 7 joints
Joints:
- joint base_head_joint: type revolute -> fixed
