Commit message: Add yaw_M3_link.

File: urdf/mira_simple_collisions_inertias.urdf (robot description, URDF)
Before this commit: robot mira, 3 links, 2 joints
Links:
- added link yaw_M3_link, mass 0.001; visual cylinder length=0.005 radius=0.01
Joints:
- added joint yaw_joint: type continuous, parent pitch_M2_link, child yaw_M3_link, origin xyz=0 0 0.01 rpy=0 0 0, axis 0 0 1, limit effort=0.1 velocity=0.01

Commit message: Base_head_link added.

File: urdf/mira_simple_collisions_inertias.urdf (robot description, URDF)
Before this commit: robot mira, 4 links, 3 joints
Links:
- added link head_link, mass 0.001; visual mesh filename=package://my_mira_description/models/mira/meshes/mira_head_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
Joints:
- added joint base_head_joint: type fixed, parent yaw_M3_link, child head_link, origin xyz=0 0 0 rpy=0 0 -1.571

Commit message: Add right and left eyes.

File: urdf/mira_simple_collisions_inertias.urdf (robot description, URDF)
Before this commit: robot mira, 5 links, 4 joints
Links:
- added link left_eye_link, mass 0.001; visual mesh filename=package://my_mira_description/models/mira/meshes/mira_eye_v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
- added link right_eye_link, mass 0.001; visual mesh filename=package://my_mira_description/models/mira/meshes/mira_eye_v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
Joints:
- added joint head_lefteye_joint: type fixed, parent head_link, child left_eye_link, origin xyz=0.0095 0.057 0.0085 rpy=-1.5708 0 0
- added joint head_righteye_joint: type fixed, parent head_link, child right_eye_link, origin xyz=-0.0095 0.057 0.0085 rpy=-1.5708 0 0

Commit message: Add camera.

File: urdf/mira_simple_collisions_inertias.urdf (robot description, URDF)
Before this commit: robot mira, 7 links, 6 joints
Links:
- added link camera_link, mass 0.001; visual box size=0.0005 0.0005 0.0005
Joints:
- added joint head_camera_joint: type fixed, parent head_link, child camera_link, origin xyz=0.0424264 0 0.0424264 rpy=0 0 0

Commit message: Add pitch and yaw controllers.

File: urdf/mira_simple_collisions_inertias.urdf (robot description, URDF)
Before this commit: robot mira, 8 links, 7 joints
Joints:
- joint yaw_joint: limit effort=0.1 velocity=0.01 -> lower=-0.2 upper=0.2 effort=0.1 velocity=0.005

Commit message: Fix position elements.

File: urdf/mira_simple_collisions_inertias.urdf (robot description, URDF)
Before this commit: robot mira, 8 links, 7 joints
Joints:
- joint base_head_joint: origin xyz=0 0 0 rpy=0 0 -1.571 -> xyz=0 0 0 rpy=0 0 0
- joint head_camera_joint: origin xyz=0.0424264 0 0.0424264 rpy=0 0 0 -> xyz=0.056507 0 0.0255139 rpy=0 0 0
- joint head_lefteye_joint: origin xyz=0.0095 0.057 0.0085 rpy=-1.5708 0 0 -> xyz=0.057 0.0095 0.0085 rpy=0 0 0
- joint head_righteye_joint: origin xyz=-0.0095 0.057 0.0085 rpy=-1.5708 0 0 -> xyz=0.057 -0.0095 0.0085 rpy=0 0 0

Commit message: Fix posistion elements.

File: urdf/mira_simple_collisions_inertias.urdf (robot description, URDF)
Before this commit: robot mira, 8 links, 7 joints
Joints:
- joint base_head_joint: origin xyz=0 0 0 rpy=0 0 0 -> xyz=0 0 0.007 rpy=0 0 0
- joint pitch_joint: limit lower=-0.2 upper=0.2 effort=0.1 velocity=0.005 -> lower=-0.17 upper=0.2 effort=0.1 velocity=0.005; origin xyz=0.0 0.0 0.0025 rpy=0 0 0 -> xyz=0.0 0.0 0.0 rpy=0 0 0
- joint roll_joint: origin xyz=0.0023 0 -0.0005 rpy=0 0 0 -> xyz=0.0023 0 0 rpy=0 0 0
- joint yaw_joint: origin xyz=0 0 0.01 rpy=0 0 0 -> xyz=0 0 0.012 rpy=0 0 0
