Commit message: Add second leg.

File: urdf/gurdy.urdf (robot description, URDF)
Before this commit: robot gurdy, 5 links, 4 joints
Links:
- added link foot_M2; visual sphere radius=0.008
- added link lower_leg_M2_link; visual cylinder length=0.06 radius=0.0015
- added link upper_leg_M2_link; visual cylinder length=0.06 radius=0.0025
Joints:
- added joint head_upper_leg_M2: type fixed, parent head_link, child upper_leg_M2_link, origin xyz=-0.026 0.0125 -0.02 rpy=0 0 0
- added joint lower_leg_M2_foot_M2: type fixed, parent lower_leg_M2_link, child foot_M2, origin xyz=0.0 0.0 -0.064 rpy=0 0 0
- added joint upper_leg_M2_lower_leg_M2: type fixed, parent upper_leg_M2_link, child lower_leg_M2_link, origin xyz=0.0 0.0 -0.06 rpy=0 0 0

Commit message: Add third leg.

File: urdf/gurdy.urdf (robot description, URDF)
Before this commit: robot gurdy, 8 links, 7 joints
Links:
- added link foot_M3; visual sphere radius=0.008
- added link lower_leg_M3_link; visual cylinder length=0.06 radius=0.0015
- added link upper_leg_M3_link; visual cylinder length=0.06 radius=0.0025
Joints:
- added joint head_upper_leg_M3: type fixed, parent head_link, child upper_leg_M3_link, origin xyz=0.0 -0.020 -0.02 rpy=0 0 0
- added joint lower_leg_M3_foot_M3: type fixed, parent lower_leg_M3_link, child foot_M3, origin xyz=0.0 0.0 -0.064 rpy=0 0 0
- added joint upper_leg_M3_lower_leg_M3: type fixed, parent upper_leg_M3_link, child lower_leg_M3_link, origin xyz=0.0 0.0 -0.06 rpy=0 0 0

Commit message: Modify position of links and joints fit dae files.

File: urdf/gurdy.urdf (robot description, URDF)
Before this commit: robot gurdy, 11 links, 10 joints
Links:
- link head_link: geometry visual mesh filename=package://my_mira_description/models/gurdy/meshes/gurdy_hea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
- link lower_leg_M1_link: geometry visual mesh filename=package://my_mira_description/models/gurdy/meshes/gurdy_low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
- link lower_leg_M2_link: geometry visual mesh filename=package://my_mira_description/models/gurdy/meshes/gurdy_low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
- link lower_leg_M3_link: geometry visual mesh filename=package://my_mira_description/models/gurdy/meshes/gurdy_low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
- link upper_leg_M1_link: geometry visual mesh filename=package://my_mira_description/models/gurdy/meshes/gurdy_hig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
- link upper_leg_M2_link: geometry visual mesh filename=package://my_mira_description/models/gurdy/meshes/gurdy_hig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
- link upper_leg_M3_link: geometry visual mesh filename=package://my_mira_description/models/gurdy/meshes/gurdy_hig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
Joints:
- joint base_head_joint: origin xyz=0.0 0.0 0.025 rpy=0 0 0 -> xyz=0.0 0.0 0.005 rpy=0 0 0
- joint head_upper_leg_M1: origin xyz=0.026 0.0125 -0.02 rpy=0 0 0 -> xyz=0.02165 -0.01250 -0.01 rpy=0 0 -0.5235
- joint head_upper_leg_M2: origin xyz=-0.026 0.0125 -0.02 rpy=0 0 0 -> xyz=-0.0225 -0.0105 -0.01 rpy=0 0 0.5235
- joint head_upper_leg_M3: origin xyz=0.0 -0.020 -0.02 rpy=0 0 0 -> xyz=0.0 0.025 -0.01 rpy=0 0 1.57079
- joint lower_leg_M1_foot_M1: origin xyz=0.0 0.0 -0.064 rpy=0 0 0 -> xyz=0.0 0.0 -0.060 rpy=0 0 0
- joint lower_leg_M2_foot_M2: origin xyz=0.0 0.0 -0.064 rpy=0 0 0 -> xyz=0.0 0.0 -0.06 rpy=0 0 0
- joint lower_leg_M3_foot_M3: origin xyz=0.0 0.0 -0.064 rpy=0 0 0 -> xyz=0.0 0.0 -0.06 rpy=0 0 0
- joint upper_leg_M2_lower_leg_M2: origin xyz=0.0 0.0 -0.06 rpy=0 0 0 -> xyz=0.0 -0.01 -0.06 rpy=0 0 0

Commit message: Change joint type to revolute, and adjust again the joints positioning.

File: urdf/gurdy.urdf (robot description, URDF)
Before this commit: robot gurdy, 11 links, 10 joints
Joints:
- joint head_upper_leg_M1: axis (none) -> 0 1 0; limit (none) -> lower=-1.5707 upper=1.5707 effort=30 velocity=1.0; origin xyz=0.02165 -0.01250 -0.01 rpy=0 0 -0.5235 -> xyz=0.02365 -0.0090359 -0.008 rpy=0 0 -0.5235; type fixed -> revolute
- joint head_upper_leg_M2: axis (none) -> 0 1 0; limit (none) -> lower=-1.5707 upper=1.5707 effort=30 velocity=1.0; origin xyz=-0.0225 -0.0105 -0.01 rpy=0 0 0.5235 -> xyz=-0.0195 -0.01569 -0.008 rpy=0 0 0.5235; type fixed -> revolute
- joint head_upper_leg_M3: axis (none) -> 0 1 0; limit (none) -> lower=-1.5707 upper=1.5707 effort=30 velocity=1.0; origin xyz=0.0 0.025 -0.01 rpy=0 0 1.57079 -> xyz=-0.004 0.025 -0.008 rpy=0 0 1.57079; type fixed -> revolute
- joint upper_leg_M1_lower_leg_M1: axis (none) -> 0 1 0; limit (none) -> lower=-1.5707 upper=1.5707 effort=30 velocity=1.0; origin xyz=0.0 0.0 -0.06 rpy=0 0 0 -> xyz=0.0 -0.006 -0.06 rpy=0 0 0; type fixed -> revolute
- joint upper_leg_M2_lower_leg_M2: axis (none) -> 0 1 0; limit (none) -> lower=-1.5707 upper=1.5707 effort=30 velocity=1.0; origin xyz=0.0 -0.01 -0.06 rpy=0 0 0 -> xyz=0.0 -0.006 -0.06 rpy=0 0 0; type fixed -> revolute
- joint upper_leg_M3_lower_leg_M3: axis (none) -> 0 1 0; limit (none) -> lower=-1.5707 upper=1.5707 effort=30 velocity=1.0; origin xyz=0.0 0.0 -0.06 rpy=0 0 0 -> xyz=0.0 -0.006 -0.06 rpy=0 0 0; type fixed -> revolute

Commit message: Add inertias & collisions to base_link.

File: urdf/gurdy.urdf (robot description, URDF)
Before this commit: robot gurdy, 11 links, 10 joints
Links:
- link base_link: mass None -> 0.001; geometry collision box size=0.01 0.01 0.01; visual box size=0.01 0.01 0.01

Commit message: Add inertias & collisions to head_link.

File: urdf/gurdy.urdf (robot description, URDF)
Before this commit: robot gurdy, 11 links, 10 joints
Links:
- link head_link: mass None -> 0.01; geometry collision cylinder length=0.04 radius=0.05; visual mesh filename=package://my_mira_description/models/gurdy/meshes/gurdy_hea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

Commit message: Add inertias & collisions to upper_leg_M1_link.

File: urdf/gurdy.urdf (robot description, URDF)
Before this commit: robot gurdy, 11 links, 10 joints
Links:
- link upper_leg_M1_link: mass None -> 0.01; geometry collision cylinder length=0.05 radius=0.003; visual mesh filename=package://my_mira_description/models/gurdy/meshes/gurdy_hig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

Commit message: Add inertias & collisions to upper_leg_M{2,3}_link.

File: urdf/gurdy.urdf (robot description, URDF)
Before this commit: robot gurdy, 11 links, 10 joints
Links:
- link upper_leg_M2_link: mass None -> 0.01; geometry collision cylinder length=0.05 radius=0.003; visual mesh filename=package://my_mira_description/models/gurdy/meshes/gurdy_hig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
- link upper_leg_M3_link: mass None -> 0.01; geometry collision cylinder length=0.05 radius=0.003; visual mesh filename=package://my_mira_description/models/gurdy/meshes/gurdy_hig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

Commit message: Add inertias & collisions to lower_M{1,2,3}_link.

File: urdf/gurdy.urdf (robot description, URDF)
Before this commit: robot gurdy, 11 links, 10 joints
Links:
- link lower_leg_M1_link: mass None -> 0.01; geometry collision cylinder length=0.04 radius=0.002; visual mesh filename=package://my_mira_description/models/gurdy/meshes/gurdy_low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
- link lower_leg_M2_link: mass None -> 0.01; geometry collision cylinder length=0.04 radius=0.002; visual mesh filename=package://my_mira_description/models/gurdy/meshes/gurdy_low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
- link lower_leg_M3_link: mass None -> 0.01; geometry collision cylinder length=0.04 radius=0.002; visual mesh filename=package://my_mira_description/models/gurdy/meshes/gurdy_low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

Commit message: Add inertias & collisions to foot_M{1,2,3}.

File: urdf/gurdy.urdf (robot description, URDF)
Before this commit: robot gurdy, 11 links, 10 joints
Links:
- link foot_M1: mass None -> 0.01; geometry collision sphere radius=0.008; visual sphere radius=0.008
- link foot_M2: mass None -> 0.01; geometry collision sphere radius=0.008; visual sphere radius=0.008
- link foot_M3: mass None -> 0.01; geometry collision sphere radius=0.008; visual sphere radius=0.008
