Commit message: Create xacros for legs and feet.

File: robot/gurdy.xacro (robot description, xacro)
@@ -27,4 +27,12 @@
   <xacro:property name="head_dim_radius" value="0.05" />
   <xacro:property name="head_dim_lenght" value="0.04" />
+  <xacro:property name="upper_leg_mass" value="0.01" />
+  <xacro:property name="upper_leg_dim_radius" value="0.003" />
+  <xacro:property name="upper_leg_dim_lenght" value="0.067" />
+  <xacro:property name="lower_leg_mass" value="0.01" />
+  <xacro:property name="lower_leg_dim_radius" value="0.002" />
+  <xacro:property name="lower_leg_dim_lenght" value="0.067" />
+  <xacro:property name="foot_mass" value="0.01" />
+  <xacro:property name="foot_radius" value="0.008" />
   <xacro:macro name="default_origin">
     <origin xyz="0 0 0" rpy="0 0 0"/>
@@ -44,4 +52,11 @@
     </inertial>
   </xacro:macro>
+  <xacro:macro name="solid_sphere_inertial" params="m r">
+    <inertial>
+      <xacro:default_origin/>
+      <mass value="${m}" />
+      <inertia ixx="${(2/5.0)*m*r*r}" ixy="0.0" ixz="0.0" iyy="${(2/5.0)*m*r*r}" iyz="0.0" izz="${(2/5.0)*m*r*r}"/>
+    </inertial>
+  </xacro:macro>
   <xacro:macro name="box_geometry" params="x y z">
     <geometry>
@@ -49,7 +64,12 @@
     </geometry>
   </xacro:macro>
-  <xacro:macro name="cylinder_geometry" params="radius lenght">
+  <xacro:macro name="cylinder_geometry" params="r l">
     <geometry>
-      <cylinder radius="${radius}" length="${lenght}" />
+      <cylinder radius="${r}" length="${l}" />
+    </geometry>
+  </xacro:macro>
+  <xacro:macro name="sphere_geometry" params="r">
+    <geometry>
+      <sphere radius="${r}"/>
     </geometry>
   </xacro:macro>
@@ -58,4 +78,50 @@
       <mesh filename="${src}" />
     </geometry>
+  </xacro:macro>
+  <xacro:macro name="leg_link" params="suffix m r l color mesh">
+    <link name="${suffix}">
+      <xacro:cylinder_inertial m="${m}" r="${r}" l="${l}">
+        <origin rpy="0.0 0.0 0.0" xyz="0 0 -0.03" />
+      </xacro:cylinder_inertial>
+      <collision>
+        <origin rpy="0.0 0.0 0.0" xyz="0 0 -0.03" />
+        <xacro:cylinder_geometry r="${r}" l="${l}"/>
+      </collision>
+      <visual>
+        <material name="${color}"/>
+        <origin xyz="0 0.0 -0.06" rpy="0 0 0"/>
+        <xacro:mesh_geometry src="${mesh}"/>
+      </visual>
+    </link>
+  </xacro:macro>
+  <xacro:macro name="leg_joint" params="suffix parent child *origin">
+    <joint name="${suffix}" type="revolute">
+      <parent link="${parent}" />
+      <child link="${child}" />
+      <xacro:insert_block name="origin"/>
+      <limit effort="30" velocity="1.0" lower="-1.5707" upper="1.5707" />
+      <axis xyz="0 1 0" />
+    </joint>
+  </xacro:macro>
+  <xacro:macro name="foot_link" params="suffix m r color">
+    <link name="${suffix}">
+      <xacro:solid_sphere_inertial m="${m}" r="${r}"/>
+      <collision>
+        <xacro:default_origin/>
+        <xacro:sphere_geometry r="${r}"/>
+      </collision>
+      <visual>
+        <material name="${color}"/>
+        <xacro:default_origin/>
+        <xacro:sphere_geometry r="${r}"/>
+      </visual>
+    </link>
+  </xacro:macro>
+  <xacro:macro name="foot_joint" params="suffix parent child">
+    <joint name="${suffix}" type="fixed">
+      <parent link="${parent}" />
+      <child link="${child}" />
+      <origin xyz="0.0 0.0 -0.060" rpy="0 0 0" />
+    </joint>
   </xacro:macro>
   <link name="base_link">
@@ -92,4 +158,14 @@
     <origin xyz="0.0 0.0 0.005" rpy="0 0 0" />
   </joint>
+  <xacro:leg_link suffix="upper_leg_M1_link" m="${upper_leg_mass}" r="${upper_leg_dim_radius}" l="${upper_leg_dim_lenght}" color="gray" mesh="package://my_mira_description/models/gurdy/meshes/gurdy_higherleg_v2.dae"/>
+  <xacro:leg_joint suffix="head_upper_leg_M1_joint" parent="head_link" child="upper_leg_M1_link">
+    <origin xyz="0.02365 -0.0090359 -0.008" rpy="0 0 -0.5235" />
+  </xacro:leg_joint>
+  <xacro:leg_link suffix="lower_leg_M1_link" m="${lower_leg_mass}" r="${lower_leg_dim_radius}" l="${lower_leg_dim_lenght}" color="gray" mesh="package://my_mira_description/models/gurdy/meshes/gurdy_lowerleg_v2.dae"/>
+  <xacro:leg_joint suffix="upper_leg_M1_lower_leg_M1_joint" parent="upper_leg_M1_link" child="lower_leg_M1_link">
+    <origin xyz="0.0 -0.006 -0.06" rpy="0 0 0" />
+  </xacro:leg_joint>
+  <xacro:foot_link suffix="foot_M1" m="${foot_mass}" r="${foot_radius}" color="blue"/>
+  <xacro:foot_joint suffix="lower_leg_M1_foot_M1_joint" parent="lower_leg_M1_link" child="foot_M1"/>
   <gazebo>
     <plugin name="gazebo_ros_control" filename="libgazebo_ros_control.so">
@@ -111,3 +187,10 @@
     <material>Gazebo/Black</material>
   </gazebo>
+  <gazebo reference="foot_M1">
+    <kp>10000.0</kp>
+    <kd>10000.0</kd>
+    <mu1>10.0</mu1>
+    <mu2>10.0</mu2>
+    <material>Gazebo/Blue</material>
+  </gazebo>
 </robot>

Commit message: Add upper 2nd and 3rd upper_leg links and joints.

File: robot/gurdy.xacro (robot description, xacro)
@@ -159,6 +159,14 @@
   </joint>
   <xacro:leg_link suffix="upper_leg_M1_link" m="${upper_leg_mass}" r="${upper_leg_dim_radius}" l="${upper_leg_dim_lenght}" color="gray" mesh="package://my_mira_description/models/gurdy/meshes/gurdy_higherleg_v2.dae"/>
+  <xacro:leg_link suffix="upper_leg_M2_link" m="${upper_leg_mass}" r="${upper_leg_dim_radius}" l="${upper_leg_dim_lenght}" color="gray" mesh="package://my_mira_description/models/gurdy/meshes/gurdy_higherleg_v2.dae"/>
+  <xacro:leg_link suffix="upper_leg_M3_link" m="${upper_leg_mass}" r="${upper_leg_dim_radius}" l="${upper_leg_dim_lenght}" color="gray" mesh="package://my_mira_description/models/gurdy/meshes/gurdy_higherleg_v2.dae"/>
   <xacro:leg_joint suffix="head_upper_leg_M1_joint" parent="head_link" child="upper_leg_M1_link">
     <origin xyz="0.02365 -0.0090359 -0.008" rpy="0 0 -0.5235" />
+  </xacro:leg_joint>
+  <xacro:leg_joint suffix="head_upper_leg_M2_joint" parent="head_link" child="upper_leg_M2_link">
+    <origin xyz="-0.0195 -0.01569 -0.008" rpy="0 0 0.5235" />
+  </xacro:leg_joint>
+  <xacro:leg_joint suffix="head_upper_leg_M3_joint" parent="head_link" child="upper_leg_M3_link">
+    <origin xyz="-0.004 0.025 -0.008" rpy="0 0 1.57079" />
   </xacro:leg_joint>
   <xacro:leg_link suffix="lower_leg_M1_link" m="${lower_leg_mass}" r="${lower_leg_dim_radius}" l="${lower_leg_dim_lenght}" color="gray" mesh="package://my_mira_description/models/gurdy/meshes/gurdy_lowerleg_v2.dae"/>

Commit message: Add lower legs and feet.

File: robot/gurdy.xacro (robot description, xacro)
@@ -161,4 +161,10 @@
   <xacro:leg_link suffix="upper_leg_M2_link" m="${upper_leg_mass}" r="${upper_leg_dim_radius}" l="${upper_leg_dim_lenght}" color="gray" mesh="package://my_mira_description/models/gurdy/meshes/gurdy_higherleg_v2.dae"/>
   <xacro:leg_link suffix="upper_leg_M3_link" m="${upper_leg_mass}" r="${upper_leg_dim_radius}" l="${upper_leg_dim_lenght}" color="gray" mesh="package://my_mira_description/models/gurdy/meshes/gurdy_higherleg_v2.dae"/>
+  <xacro:leg_link suffix="lower_leg_M1_link" m="${lower_leg_mass}" r="${lower_leg_dim_radius}" l="${lower_leg_dim_lenght}" color="gray" mesh="package://my_mira_description/models/gurdy/meshes/gurdy_lowerleg_v2.dae"/>
+  <xacro:leg_link suffix="lower_leg_M2_link" m="${lower_leg_mass}" r="${lower_leg_dim_radius}" l="${lower_leg_dim_lenght}" color="gray" mesh="package://my_mira_description/models/gurdy/meshes/gurdy_lowerleg_v2.dae"/>
+  <xacro:leg_link suffix="lower_leg_M3_link" m="${lower_leg_mass}" r="${lower_leg_dim_radius}" l="${lower_leg_dim_lenght}" color="gray" mesh="package://my_mira_description/models/gurdy/meshes/gurdy_lowerleg_v2.dae"/>
+  <xacro:foot_link suffix="foot_M1" m="${foot_mass}" r="${foot_radius}" color="blue"/>
+  <xacro:foot_link suffix="foot_M2" m="${foot_mass}" r="${foot_radius}" color="green"/>
+  <xacro:foot_link suffix="foot_M3" m="${foot_mass}" r="${foot_radius}" color="red"/>
   <xacro:leg_joint suffix="head_upper_leg_M1_joint" parent="head_link" child="upper_leg_M1_link">
     <origin xyz="0.02365 -0.0090359 -0.008" rpy="0 0 -0.5235" />
@@ -170,10 +176,16 @@
     <origin xyz="-0.004 0.025 -0.008" rpy="0 0 1.57079" />
   </xacro:leg_joint>
-  <xacro:leg_link suffix="lower_leg_M1_link" m="${lower_leg_mass}" r="${lower_leg_dim_radius}" l="${lower_leg_dim_lenght}" color="gray" mesh="package://my_mira_description/models/gurdy/meshes/gurdy_lowerleg_v2.dae"/>
   <xacro:leg_joint suffix="upper_leg_M1_lower_leg_M1_joint" parent="upper_leg_M1_link" child="lower_leg_M1_link">
     <origin xyz="0.0 -0.006 -0.06" rpy="0 0 0" />
   </xacro:leg_joint>
-  <xacro:foot_link suffix="foot_M1" m="${foot_mass}" r="${foot_radius}" color="blue"/>
+  <xacro:leg_joint suffix="upper_leg_M2_lower_leg_M2_joint" parent="upper_leg_M2_link" child="lower_leg_M2_link">
+    <origin xyz="0.0 -0.006 -0.06" rpy="0 0 0" />
+  </xacro:leg_joint>
+  <xacro:leg_joint suffix="upper_leg_M3_lower_leg_M3_joint" parent="upper_leg_M3_link" child="lower_leg_M3_link">
+    <origin xyz="0.0 -0.006 -0.06" rpy="0 0 0" />
+  </xacro:leg_joint>
   <xacro:foot_joint suffix="lower_leg_M1_foot_M1_joint" parent="lower_leg_M1_link" child="foot_M1"/>
+  <xacro:foot_joint suffix="lower_leg_M2_foot_M2_joint" parent="lower_leg_M2_link" child="foot_M2"/>
+  <xacro:foot_joint suffix="lower_leg_M3_foot_M3_joint" parent="lower_leg_M3_link" child="foot_M3"/>
   <gazebo>
     <plugin name="gazebo_ros_control" filename="libgazebo_ros_control.so">
@@ -197,10 +209,15 @@
     <material>Gazebo/Black</material>
   </gazebo>
-  <gazebo reference="foot_M1">
-    <kp>10000.0</kp>
-    <kd>10000.0</kd>
-    <mu1>10.0</mu1>
-    <mu2>10.0</mu2>
-    <material>Gazebo/Blue</material>
-  </gazebo>
+  <xacro:macro name="gazebo_reference_foot" params="ref color">
+    <gazebo reference="${ref}">
+      <kp>10000.0</kp>
+      <kd>10000.0</kd>
+      <mu1>10.0</mu1>
+      <mu2>10.0</mu2>
+      <material>Gazebo/${color}</material>
+    </gazebo>
+  </xacro:macro>
+  <xacro:gazebo_reference_foot ref="foot_M1" color="Blue"/>
+  <xacro:gazebo_reference_foot ref="foot_M2" color="Green"/>
+  <xacro:gazebo_reference_foot ref="foot_M3" color="Red"/>
 </robot>

Commit message: Create xacro macro for gazebo reference upper legs.

File: robot/gurdy.xacro (robot description, xacro)
@@ -218,4 +218,16 @@
     </gazebo>
   </xacro:macro>
+  <xacro:macro name="gazebo_reference_upper_leg" params="ref color">
+    <gazebo reference="${ref}">
+      <kp>10000.0</kp>
+      <kd>10000.0</kd>
+      <mu1>10.0</mu1>
+      <mu2>10.0</mu2>
+      <material>Gazebo/${color}</material>
+    </gazebo>
+  </xacro:macro>
+  <xacro:gazebo_reference_upper_leg ref="upper_leg_M1_link" color="Black"/>
+  <xacro:gazebo_reference_upper_leg ref="upper_leg_M2_link" color="Black"/>
+  <xacro:gazebo_reference_upper_leg ref="upper_leg_M3_link" color="Black"/>
   <xacro:gazebo_reference_foot ref="foot_M1" color="Blue"/>
   <xacro:gazebo_reference_foot ref="foot_M2" color="Green"/>

Commit message: Create xacro for transmissions.

File: robot/gurdy.xacro (robot description, xacro)
@@ -124,4 +124,16 @@
       <origin xyz="0.0 0.0 -0.060" rpy="0 0 0" />
     </joint>
+  </xacro:macro>
+  <xacro:macro name="revolute_trans" params="trans_name type joint_name act_name hw_inter reduc">
+    <transmission name="${trans_name}">
+        <type>${type}</type>
+        <joint name="${joint_name}">
+            <hardwareInterface>${hw_inter}</hardwareInterface>
+        </joint>
+        <actuator name="${act_name}">
+            <hardwareInterface>${hw_inter}</hardwareInterface>
+            <mechanicalReduction>${reduc}</mechanicalReduction>
+        </actuator>
+    </transmission>
   </xacro:macro>
   <link name="base_link">
@@ -188,4 +200,10 @@
   <xacro:foot_joint suffix="lower_leg_M2_foot_M2_joint" parent="lower_leg_M2_link" child="foot_M2"/>
   <xacro:foot_joint suffix="lower_leg_M3_foot_M3_joint" parent="lower_leg_M3_link" child="foot_M3"/>
+  <xacro:revolute_trans trans_name="trans1" type="transmission_interface/SimpleTransmission" joint_name="head_upper_leg_M1_joint" act_name="motor1" hw_inter="hardware_interface/EffortJointInterface" reduc="1"/>
+  <xacro:revolute_trans trans_name="trans2" type="transmission_interface/SimpleTransmission" joint_name="upper_leg_M1_lower_leg_M1_joint" act_name="motor2" hw_inter="hardware_interface/EffortJointInterface" reduc="1"/>
+  <xacro:revolute_trans trans_name="trans3" type="transmission_interface/SimpleTransmission" joint_name="head_upper_leg_M2_joint" act_name="motor3" hw_inter="hardware_interface/EffortJointInterface" reduc="1"/>
+  <xacro:revolute_trans trans_name="trans4" type="transmission_interface/SimpleTransmission" joint_name="upper_leg_M2_lower_leg_M2_joint" act_name="motor4" hw_inter="hardware_interface/EffortJointInterface" reduc="1"/>
+  <xacro:revolute_trans trans_name="trans5" type="transmission_interface/SimpleTransmission" joint_name="head_upper_leg_M3_joint" act_name="motor5" hw_inter="hardware_interface/EffortJointInterface" reduc="1"/>
+  <xacro:revolute_trans trans_name="trans6" type="transmission_interface/SimpleTransmission" joint_name="upper_leg_M3_lower_leg_M3_joint" act_name="motor6" hw_inter="hardware_interface/EffortJointInterface" reduc="1"/>
   <gazebo>
     <plugin name="gazebo_ros_control" filename="libgazebo_ros_control.so">
